File: PCB/project.kicad_pcb (KiCad board)
At the start: 2 copper layers, 146.1 x 73.8 mm, 69 parts, among them J1 UART, J2 SWD, J4 Conn_01x10, K1 Компрессор, K2 ТЕН поддон, K3 ТЕН компрессор, Q1 IRLML0030, Q2 IRLML0030, Q3 IRLML0030, Q4 IRLML0030, U1 STM32F030F4Px, U2 EL814, U3 EL814, U4 12->3.3, U5 TL431AID, Y1 8MHz

Commit message: PCB and schematic done
Parts:
- added H1: MountingHole, MountingHole:MountingHole_3.2mm_M3, F.Cu at (76.7, 49.4)
- added H2: MountingHole, MountingHole:MountingHole_3.2mm_M3, F.Cu at (76.6, 127.7)
- added H3: MountingHole, MountingHole:MountingHole_3.2mm_M3, F.Cu at (166.1, 49.2)
- added H4: MountingHole, MountingHole:MountingHole_3.2mm_M3, F.Cu at (166.2, 128.0)
- C12: renamed from C14; moved to B.Cu
- C15: renamed from C13; moved to B.Cu
- C5: renamed from C12; value 100nF -> 100pF
- C6: renamed from C8; value 100nF -> 10uF
- C7: moved to B.Cu
- C9: renamed from C10; moved to B.Cu
- J3: renamed from J4; footprint Connector_Phoenix_MSTB:PhoenixContact_MSTBA_2,5_10-G_1x10_P5.00mm_Horizontal -> Connector_Phoenix_MSTB:PhoenixContact_MSTB_2,5_10-GF-5,08_1x10_P5.08mm_Horizontal_ThreadedFlange
- K2: value ТЕН поддон -> Relay_SPST-NO; footprint Relay_THT:Relay_SPDT_Hongfa_HF3F-L-xx-1ZL1T -> Relay_THT:Relay_SPST_Schrack-RP-II-1-FormA_RM3.5mm
- K3: value ТЕН компрессор -> Relay_SPST-NO; footprint Relay_THT:Relay_SPDT_Hongfa_HF3F-L-xx-1ZL1T -> Relay_THT:Relay_SPST_Schrack-RP-II-1-FormA_RM3.5mm
- PS1: value HLK-10M12 -> HLK-PM12; footprint Converter_ACDC:Converter_ACDC_Hi-Link_HLK-10Mxx -> Converter_ACDC:Converter_ACDC_Hi-Link_HLK-PMxx
- Q1: renamed from Q4; moved to B.Cu
- R10: renamed from R21; moved to B.Cu
- R11: renamed from R22; moved to B.Cu
- R12: renamed from R6; moved to B.Cu
- R13: renamed from R7; moved to B.Cu
- R14: renamed from R10; moved to B.Cu
- R18: renamed from R5; moved to B.Cu
- R19: renamed from R8; moved to B.Cu
- R20: renamed from R11; moved to B.Cu
- R24: renamed from R3; moved to B.Cu
- R25: renamed from R4; moved to B.Cu
- R7: renamed from R14; moved to B.Cu
- R8: renamed from R18; moved to B.Cu
- R9: renamed from R20; moved to B.Cu
- moved U1 139.8 mm to (133.7, 67.0)
- moved R18 132.8 mm to (107.1, 54.1)
- moved C7 129.5 mm to (128.2, 53.5)
- moved C9 126.7 mm to (133.9, 53.5), turned to 180 degrees
- moved C5 126.0 mm to (133.6, 63.1)
- moved R3 125.7 mm to (128.5, 62.8)
- moved R5 124.9 mm to (129.3, 66.8), turned to 90 degrees
- moved R6 120.6 mm to (133.6, 70.5), turned to 180 degrees
- moved C15 118.6 mm to (146.8, 122.8)
- moved C8 116.8 mm to (127.0, 56.0)
- moved U3 114.7 mm to (128.5, 50.4)
- moved C12 112.7 mm to (152.1, 122.8)
- moved C2 111.8 mm to (151.6, 55.9)
- moved R19 111.7 mm to (127.7, 77.2)
- moved J1 108.8 mm to (158.4, 63.1), turned to 90 degrees
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- renumbered C5 to C1, C11 to C10, C3 to C11, C1 to C13, C2 to C14, C15 to C2, C4 to C3, C6 to C4, C9 to C8, D4 to D1, D5 to D2, D6 to D3, D7 to D4, D1 to D5, D2 to D6, D3 to D7, Q1 to Q2, Q2 to Q3, Q3 to Q4, R13 to R1, R23 to R15, R24 to R16, R25 to R17, R12 to R2, R9 to R21, R1 to R22, R2 to R23, R15 to R3, R19 to R4, R16 to R5, R17 to R6, U5 to U1, U1 to U2, U4 to U3, U2 to U4, U3 to U5
Connections:
- F1 pad 1: 220 вход (L) -> 220 вход (N)
- J3 pad 1: 220 вход (N) -> 220 вход (L)
- J3 pad 2: 220 вход (L) -> 220 вход (N)
- R22 pad 1: 220 вход (N) -> Net-(F2-Pad2)
- R23 pad 1: 220 вход (N) -> Net-(F3-Pad2)
- TH1 pad 1: 220 вход (N) -> 220 вход (L)
- U2 pad 11: компрессор упр. -> ТЕН поддон упр.
- U2 pad 12: ТЕН поддон упр. -> компрессор упр.
- U4 pad 2: Net-(F2-Pad2) -> 220 вход (N)
- U5 pad 2: Net-(F3-Pad2) -> 220 вход (N)
Routing:
- net +12V: track 38.0 -> 172.8 mm, vias 0 -> 1
- net NTC темп. компрессор: track 0.00 -> 107.3 mm, vias 0 -> 2
- net NTC темп. внешняя: track 0.00 -> 101.0 mm, vias 0 -> 2
- net GND: track 0.00 -> 72.5 mm, vias 0 -> 2
- net +3V3: track 17.9 -> 72.7 mm, vias 0 -> 2
- net Net-(Q2-G): track 0.00 -> 45.6 mm
- net 4х ходовой статус: track 5.67 -> 47.7 mm, vias 0 -> 1
- net VDDA: track 7.79 -> 49.1 mm, vias 0 -> 1
- net компрессор статус: track 5.54 -> 42.2 mm, vias 0 -> 1
- net Net-(Q3-G): track 0.00 -> 27.8 mm, vias 0 -> 2
- net 220 вход (N): track 104.2 -> 128.6 mm
- net 220 тен комп. выход (L): track 50.9 -> 27.8 mm
- net Net-(Q4-G): track 0.00 -> 21.8 mm, vias 0 -> 2
- net Net-(PS1-AC/L): track 27.6 -> 7.86 mm
- net 220 комп. вход (L): track 43.2 -> 24.5 mm
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- added copper zone on B.Cu, net GND
Other:
- board size 146.1 x 73.8 mm -> 98.1 x 87.7 mm
- board text added: "1"
- board text added: "1 - Компресор фаза 2 - ТЕН піддон 3 - ТЕН компресор 4 - Компресор вхід 5 - 4х ход. вхід 6 - Темп. компресор 7 - Темп. зовнішня 8 - Темп. загальний"
- board text added: "2"
- board text added: "3"
- board text added: "3v3"
- board text added: "4"
- board text added: "5"
- board text added: "6"
- board text added: "7"
- board text added: "8"
- board text added: "CLK"
- board text added: "DIO"
- board text added: "EVK 2025 rev 1.0"
- board text added: "GND"
- board text added: "JLCJLCJLCJLC"
- board text added: "L"
- board text added: "N"
- board text added: "RST"
- board text added: "RX"
- board text added: "SWD"
- board text added: "TX"
- board text added: "UART"
- board text added: "Компресор"
- board text added: "Прилад керування обігрівом зовнішнього блоку"
- board text added: "Режим"
- board text added: "ТЕН Компр."
- board text added: "ТЕН Піддон"
